Commit message: corrected some package namespace issues from files copied over from shelly.pkg

File: urdf/shelly.xacro (robot description, xacro)
@@ -110,5 +110,5 @@
  <!-- ################### ROBOT Definitions ############################# -->
 <!--Includes Sensor Plugins defined in .gazebo file-->
-<xacro:include filename="$(find shelly)/urdf/shelly.gazebo" />
+<xacro:include filename="$(find rtab)/urdf/shelly.gazebo" />
 <link name="robot_footprint"></link>
   <joint name="robot_footprint_joint" type="fixed">
@@ -138,5 +138,5 @@
             <!--<box size=".4 .2 .1"/>-->
             <!-- <cylinder radius="0.1" length="0.4"/> -->
-            <mesh filename="package://shelly/models/meshes/green_shell.dae"/>
+            <mesh filename="package://rtab/models/meshes/green_shell.dae"/>
         </geometry>
     </visual>
@@ -263,5 +263,5 @@
             <!--
             <geometry>
-                <mesh filename="package://shelly/models/meshes/hokuyo.dae"/>
+                <mesh filename="package://rtab/models/meshes/hokuyo.dae"/>
             </geometry>
             -->

Commit message: solved xacro spawn name errors

File: urdf/shelly.xacro (robot description, xacro)
@@ -138,5 +138,5 @@
             <!--<box size=".4 .2 .1"/>-->
             <!-- <cylinder radius="0.1" length="0.4"/> -->
-            <mesh filename="package://rtab/models/meshes/green_shell.dae"/>
+            <mesh filename="package://rtab/models/green_shell.dae"/>
         </geometry>
     </visual>
@@ -236,5 +236,5 @@
             <xacro:zero_origin/>
             <geometry>
-                <mesh filename="package://rtab/kinect/meshes/kinect.dae"/>
+                <mesh filename="package://rtab/models/kinect/meshes/kinect.dae"/>
             </geometry>
             <!--<xacro:generate_geometry shape="box" x="0.05" y="0.05" z="0.05"/>-->

Commit message: was getting tf errors with the camera links, so as per rtabmap forum, Icorrected camera tf subtree. camera_link now has two sub trees, camera_rgb and camera_depth and each has their optical subtree

File: urdf/shelly.xacro (robot description, xacro)
@@ -222,5 +222,5 @@
     <!--    <child link="camera"/>-->
     <!--</joint>-->
-    <link name="kinect">
+    <link name="camera_link">
         <inertial>
             <xacro:zero_origin/>
@@ -231,5 +231,5 @@
         <collision>
             <xacro:zero_origin/>
-            <xacro:generate_geometry shape="box" x="0.05" y="0.05" z="0.05"/>
+            <xacro:generate_geometry shape="box" x="0.07" y="0.3" z="0.069"/>
         </collision>
         <visual>
@@ -245,6 +245,34 @@
         <origin xyz="0.2 0 0" rpy="0 0 0"/>
         <parent link="chassis"/>
-        <child link="kinect"/>
-    </joint>
+        <child link="camera_link"/>
+    </joint>
+    <!-- Kinect RGB Camera Frame -->
+    <link name="camera_rgb_frame"/>
+    <joint name="camera_rgb_joint" type="fixed">
+      <origin xyz="0 0 0" rpy="-1.571 0 -1.571"/>
+      <parent link="camera_link"/>
+      <child link="camera_rgb_frame"/>
+    </joint>
+        <!-- Kinect RGB Camera Optical Frame -->
+        <link name="camera_rgb_optical_frame"/>
+        <joint name="camera_rgb_optical_joint" type="fixed">
+          <origin xyz="0 0 0" rpy="-1.571 0 -1.571"/>
+          <parent link="camera_rgb_frame"/>
+          <child link="camera_rgb_optical_frame"/>
+        </joint>
+    <!-- Kinect Depth Camera Frame -->
+    <link name="camera_depth_frame"/>
+    <joint name="camera_depth_joint" type="fixed">
+      <origin xyz="0 0 0" rpy="0 0 0"/>
+      <parent link="camera_link"/>
+      <child link="camera_depth_frame"/>
+    </joint>
+        <!-- Kinect Depth Camera Optical Frame -->
+        <link name="camera_depth_optical_frame"/>
+        <joint name="camera_depth_optical_joint" type="fixed">
+          <origin xyz="0 0 0" rpy="-1.571 0 -1.571"/>
+          <parent link="camera_depth_frame"/>
+          <child link="camera_depth_optical_frame"/>
+        </joint>
     <link name="hokuyo">
         <inertial>

Commit message: the tf tree seems to match correctly, but im still getting the error in THIS_ERROR.txt, because the camera topics are being published with double prefixes, /camera/camera

File: urdf/shelly.xacro (robot description, xacro)
@@ -222,5 +222,6 @@
     <!--    <child link="camera"/>-->
     <!--</joint>-->
-    <link name="camera_link">
+    <!--<link name="camera_link">-->
+    <link name="camera_rgb_frame">
         <inertial>
             <xacro:zero_origin/>
@@ -245,7 +246,8 @@
         <origin xyz="0.2 0 0" rpy="0 0 0"/>
         <parent link="chassis"/>
-        <child link="camera_link"/>
-    </joint>
-    <!-- Kinect RGB Camera Frame -->
+        <!--<child link="camera_link"/>-->
+        <child link="camera_rgb_frame"/>
+    </joint>
+    <!-- Kinect RGB Camera Frame
     <link name="camera_rgb_frame"/>
     <joint name="camera_rgb_joint" type="fixed">
@@ -254,4 +256,5 @@
       <child link="camera_rgb_frame"/>
     </joint>
+-->
         <!-- Kinect RGB Camera Optical Frame -->
         <link name="camera_rgb_optical_frame"/>
@@ -265,5 +268,6 @@
     <joint name="camera_depth_joint" type="fixed">
       <origin xyz="0 0 0" rpy="0 0 0"/>
-      <parent link="camera_link"/>
+      <!-- <parent link="camera_link"/> -->
+      <parent link="camera_rgb_frame"/>
       <child link="camera_depth_frame"/>
     </joint>

Commit message: forgot the '/' prefix on the camera topic names. the error hasn't stopped, but its no longer fatal, and it is now attempting to map

File: urdf/shelly.xacro (robot description, xacro)
@@ -110,5 +110,5 @@
  <!-- ################### ROBOT Definitions ############################# -->
 <!--Includes Sensor Plugins defined in .gazebo file-->
-<xacro:include filename="$(find rtab)/urdf/shelly.gazebo" />
+<xacro:include filename="$(find rtab_shelly)/urdf/shelly.gazebo" />
 <link name="robot_footprint"></link>
   <joint name="robot_footprint_joint" type="fixed">
@@ -137,6 +137,6 @@
         <geometry>
             <!--<box size=".4 .2 .1"/>-->
-            <!-- <cylinder radius="0.1" length="0.4"/> -->
-            <mesh filename="package://rtab/models/green_shell.dae"/>
+            <cylinder radius="0.1" length="0.4"/>
+            <!-- <mesh filename="package://rtab_shelly/models/green_shell.dae"/> -->
         </geometry>
     </visual>
@@ -237,5 +237,5 @@
             <xacro:zero_origin/>
             <geometry>
-                <mesh filename="package://rtab/models/kinect/meshes/kinect.dae"/>
+                <mesh filename="package://rtab_shelly/models/kinect/meshes/kinect.dae"/>
             </geometry>
             <!--<xacro:generate_geometry shape="box" x="0.05" y="0.05" z="0.05"/>-->
@@ -295,5 +295,5 @@
             <!--
             <geometry>
-                <mesh filename="package://rtab/models/meshes/hokuyo.dae"/>
+                <mesh filename="package://rtab_shelly/models/meshes/hokuyo.dae"/>
             </geometry>
             -->

Commit message: reduced weight to allow easier teleop control

File: urdf/shelly.xacro (robot description, xacro)
@@ -121,5 +121,6 @@
       <pose>0 0 0 0 0 0</pose>
       <inertial>
-          <mass value="15.0"/>
+          <!--<mass value="15.0"/>-->
+          <mass value="1.0"/>
           <origin xyz="0.0 0 0" rpy=" 0 0 0"/>
           <!--  <xacro:default_inertia/> -->
@@ -134,5 +135,6 @@
     </collision>
     <visual name='chassis_visual'>
-        <xacro:shell_origin/>
+        <!--<xacro:shell_origin/>-->
+        <xacro:cylinder_origin/>
         <geometry>
             <!--<box size=".4 .2 .1"/>-->

Commit message: successfully mapped kitchen world, took screenshots of the loop closures and of the resulting point cloud

File: urdf/shelly.xacro (robot description, xacro)
@@ -246,5 +246,5 @@
     </link>
     <joint name="camera_joint" type="fixed">
-        <origin xyz="0.2 0 0" rpy="0 0 0"/>
+        <origin xyz="0.28 0 0.1" rpy="0 0 0"/>
         <parent link="chassis"/>
         <!--<child link="camera_link"/>-->
@@ -303,5 +303,5 @@
     </link>
     <joint name="hokuyo_joint" type="fixed">
-        <origin xyz="0.15 0 0.15" rpy="0 0 0"/>
+        <origin xyz="0 0 0.2" rpy="0 0 0"/>
         <parent link="chassis"/>
         <child link="hokuyo"/>

Commit message: photo shoot of each step building the world

File: urdf/shelly.xacro (robot description, xacro)
@@ -136,9 +136,9 @@
     <visual name='chassis_visual'>
         <!--<xacro:shell_origin/>-->
-        <xacro:cylinder_origin/>
+        <xacro:shell_origin/>
         <geometry>
             <!--<box size=".4 .2 .1"/>-->
-            <cylinder radius="0.1" length="0.4"/>
-            <!-- <mesh filename="package://rtab_shelly/models/green_shell.dae"/> -->
+            <!--<cylinder radius="0.1" length="0.4"/>-->
+            <mesh filename="package://rtab_shelly/models/green_shell.dae"/>
         </geometry>
     </visual>
@@ -290,18 +290,15 @@
         <collision>
             <xacro:zero_origin/>
-            <xacro:generate_geometry shape="box" x="0.1" y="0.1" z="0.1"/>
+            <xacro:generate_geometry shape="box" x="0.01" y="0.01" z="0.01"/>
         </collision>
         <visual>
             <xacro:zero_origin/>
-            <xacro:generate_geometry shape="sphere" radius="0.001"/>
-            <!--
             <geometry>
-                <mesh filename="package://rtab_shelly/models/meshes/hokuyo.dae"/>
+                <mesh filename="package://rtab_shelly/models/hokuyo.dae"/>
             </geometry>
-            -->
         </visual>
     </link>
     <joint name="hokuyo_joint" type="fixed">
-        <origin xyz="0 0 0.2" rpy="0 0 0"/>
+        <origin xyz="0 0 0.3" rpy="0 0 0"/> <!-- for shell -->
         <parent link="chassis"/>
         <child link="hokuyo"/>
